File: ECB.kicad_sch (KiCad schematic)
At the start: 5 parts, among them U2 74LS08, U5 74LS245, U6 C96ABC, U7 74LS244

Commit message: V1.1
Connections:
- net B_A3: now also U7.11 (I0b)
- net B_A4: now also U7.8 (I3a)
- net A4: now reaches U7.12 (O3a)
- net A3: now reaches U7.9 (O0b)
- no-connect marks 69 -> 65
Changed lines of the file:
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@@
 	(generator_version "9.0")
 	(paper "A4")
+	(title_block
+		(date "2026-10-24")
+		(rev "V1.1")
+	)
 	(junction
 		(at 26.67 52.07)
@@
 	)
 	(no_connect
-		(at 138.43 123.19)
-	)
-	(no_connect
 		(at 153.67 38.1)
 	)
@@
 	)
 	(no_connect
-		(at 138.43 125.73)
-	)
-	(no_connect
 		(at 115.57 38.1)
 	)
@@
 	)
 	(no_connect
-		(at 163.83 125.73)
-	)
-	(no_connect
 		(at 176.53 38.1)
 	)
@@
 	)
 	(no_connect
-		(at 163.83 123.19)
-	)
-	(no_connect
 		(at 105.41 38.1)
 	)
@@
 	)
 	(no_connect
-		(at 133.35 38.1)
+		(at 181.61 38.1)
 	)
 	(no_connect
@@
 	(wire
 		(pts
+			(xy 125.73 125.73) (xy 138.43 125.73)
+		)
+		(stroke
+			(width 0)
+			(type default)
+		)
+	)
+	(wire
+		(pts
 			(xy 194.31 45.72) (xy 194.31 38.1)
 		)
@@
 	(wire
 		(pts
+			(xy 163.83 123.19) (xy 176.53 123.19)
+		)
+		(stroke
+			(width 0)
+			(type default)
+		)
+	)
+	(wire
+		(pts
 			(xy 245.11 71.12) (xy 245.11 38.1)
 		)
@@
 	(wire
 		(pts
+			(xy 163.83 125.73) (xy 176.53 125.73)
+		)
+		(stroke
+			(width 0)
+			(type default)
+		)
+	)
+	(wire
+		(pts
 			(xy 31.75 38.1) (xy 31.75 71.12)
 		)
@@
 	(wire
 		(pts
+			(xy 125.73 123.19) (xy 138.43 123.19)
+		)
+		(stroke
+			(width 0)
+			(type default)
+		)
+	)
+	(wire
+		(pts
 			(xy 125.73 118.11) (xy 138.43 118.11)
 		)
@@
 		)
 	)
+	(global_label "B_A4"
+		(shape input)
+		(at 125.73 123.19 180)
+		(fields_autoplaced yes)
+		(effects
+			(font
+				(size 1.27 1.27)
+			)
+			(justify right)
+		)
+		(property "Intersheetrefs" "${INTERSHEET_REFS}"
+			(at 118.2091 123.19 0)
+			(effects
+				(font
+					(size 1.27 1.27)
+				)
+				(justify right)
+				(hide yes)
+			)
+		)
+	)
 	(global_label "B_DT/R"
 		(shape output)
@@
 		)
 	)
+	(global_label "A3"
+		(shape output)
+		(at 176.53 125.73 0)
+		(fields_autoplaced yes)
+		(effects
+			(font
+				(size 1.27 1.27)
+			)
+			(justify left)
+		)
+		(property "Intersheetrefs" "${INTERSHEET_REFS}"
+			(at 181.8133 125.73 0)
+			(effects
+				(font
+					(size 1.27 1.27)
+				)
+				(justify left)
+				(hide yes)
+			)
+		)
+	)
 	(global_label "B_~{IR7}"
 		(shape input)
@@
 		)
 	)
+	(global_label "A4"
+		(shape output)
+		(at 176.53 123.19 0)
+		(fields_autoplaced yes)
+		(effects
+			(font
+				(size 1.27 1.27)
+			)
+			(justify left)
+		)
+		(property "Intersheetrefs" "${INTERSHEET_REFS}"
+			(at 181.8133 123.19 0)
+			(effects
+				(font
+					(size 1.27 1.27)
+				)
+				(justify left)
+				(hide yes)
+			)
+		)
+	)
 	(global_label "B_A0"
 		(shape input)
@@
 			(effects
 				(font
+					(size 1.27 1.27)
+				)
+				(justify right)
+				(hide yes)
+			)
+		)
+	)
+	(global_label "B_A3"
+		(shape input)
+		(at 125.73 125.73 180)
+		(fields_autoplaced yes)
+		(effects
+			(font
+				(size 1.27 1.27)
+			)
+			(justify right)
+		)
+		(property "Intersheetrefs" "${INTERSHEET_REFS}"
+			(at 118.2091 125.73 0)
+			(effects
+				(font
