File: Keyboard.kicad_sch (KiCad schematic)
At the start: 8 parts, among them K1 INTERRUPT SELECT, P6 8 MHz, P7 MOUSE, P8 KEYBOARD, P9 IO PORT, U1 74LS04, U4 74LS32

Commit message: V1.1
Parts:
- removed unit 3 of U1
- U1: value 74LS04 -> 74LS06
Connections:
- net PU1: now reaches K1.2 (Pin_2)
- net PU1: now also U1.4
- net B_~{INT} renamed B_/IR6
Changed lines of the file:
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@@
 	(generator_version "9.0")
 	(paper "A4")
+	(title_block
+		(date "2026-10-24")
+		(rev "V1.1")
+	)
 	(text "KEYBOARD AND MOUSE"
 		(exclude_from_sim no)
@@
 	)
 	(junction
+		(at 106.68 125.73)
+		(diameter 0)
+		(color 0 0 0 0)
+	)
+	(junction
 		(at 33.02 46.99)
 		(diameter 0)
@@
 	(wire
 		(pts
-			(xy 104.14 125.73) (xy 109.22 125.73)
+			(xy 104.14 125.73) (xy 106.68 125.73)
 		)
 		(stroke
@@
 	(wire
 		(pts
+			(xy 106.68 125.73) (xy 132.08 125.73)
+		)
+		(stroke
+			(width 0)
+			(type default)
+		)
+	)
+	(wire
+		(pts
 			(xy 181.61 63.5) (xy 182.88 63.5)
 		)
@@
 	(wire
 		(pts
-			(xy 132.08 125.73) (xy 124.46 125.73)
-		)
-		(stroke
-			(width 0)
-			(type default)
-		)
-	)
-	(wire
-		(pts
 			(xy 154.94 90.17) (xy 154.94 100.33)
 		)
@@
 	(wire
 		(pts
+			(xy 106.68 133.35) (xy 104.14 133.35)
+		)
+		(stroke
+			(width 0)
+			(type default)
+		)
+	)
+	(wire
+		(pts
+			(xy 106.68 125.73) (xy 106.68 133.35)
+		)
+		(stroke
+			(width 0)
+			(type default)
+		)
+	)
+	(wire
+		(pts
 			(xy 128.27 72.39) (xy 129.54 72.39)
 		)
@@
 		)
 	)
+	(global_label "B_{slash}IR6"
+		(shape output)
+		(at 137.16 118.11 0)
+		(fields_autoplaced yes)
+		(effects
+			(font
+				(size 1.27 1.27)
+			)
+			(justify left)
+		)
+		(property "Intersheetrefs" "${INTERSHEET_REFS}"
+			(at 148.5151 118.11 0)
+			(effects
+				(font
+					(size 1.27 1.27)
+				)
+				(justify left)
+				(hide yes)
+			)
+		)
+	)
 	(global_label "P14"
 		(shape bidirectional)
@@
 		)
 	)
+	(global_label "PU1"
+		(shape input)
+		(at 104.14 133.35 180)
+		(fields_autoplaced yes)
+		(effects
+			(font
+				(size 1.27 1.27)
+			)
+			(justify right)
+		)
+		(property "Intersheetrefs" "${INTERSHEET_REFS}"
+			(at 97.3448 133.35 0)
+			(effects
+				(font
+					(size 1.27 1.27)
+				)
+				(justify right)
+				(hide yes)
+			)
+		)
+	)
 	(global_label "D1"
 		(shape bidirectional)
@@
 		)
 	)
-	(global_label "B_~{INT}"
-		(shape output)
-		(at 137.16 118.11 0)
-		(fields_autoplaced yes)
-		(effects
-			(font
-				(size 1.27 1.27)
-			)
-			(justify left)
-		)
-		(property "Intersheetrefs" "${INTERSHEET_REFS}"
-			(at 148.3337 118.11 0)
-			(effects
-				(font
-					(size 1.27 1.27)
-				)
-				(justify left)
-				(hide yes)
-			)
-		)
-	)
 	(symbol
 		(lib_id "Custom:DIL14")
@@
 			)
 		)
-		(property "Value" "74LS04"
+		(property "Value" "74LS06"
 			(at 178.816 66.675 0)
 			(effects
@@
 			)
 		)
-		(property "Value" "74LS04"
+		(property "Value" "74LS06"
 			(at 178.816 103.505 0)
 			(effects
@@
 			)
 		)
-		(property "Value" "74LS04"
+		(property "Value" "74LS06"
 			(at 178.816 55.245 0)
 			(effects
@@
 			)
 		)
-		(property "Value" "74LS04"
+		(property "Value" "74LS06"
 			(at 178.816 92.075 0)
 			(effects
@@
 	)
 	(symbol
-		(lib_id "74xx:74LS04")
-		(at 116.84 125.73 0)
-		(unit 3)
-		(exclude_from_sim no)
-		(in_bom yes)
-		(on_board yes)
-		(dnp no)
-		(property "Reference" "U1"
-			(at 115.824 125.984 0)
-			(effects
-				(font
-					(size 1.524 1.524)
-				)
-			)
-		)
-		(property "Value" "74LS04"
-			(at 121.666 128.905 0)
-			(effects
-				(font
-					(size 1.524 1.524)
-				)
-			)
-		)
-		(property "Footprint" "Custom:STD_DDW_DIP14"
-			(at 116.84 125.73 0)
-			(effects
-				(font
-					(size 1.27 1.27)
-				)
-				(hide yes)
-			)
-		)
-		(property "Datasheet" "http://www.ti.com/lit/gpn/sn74LS04"
-			(at 116.84 125.73 0)
-			(effects
-				(font
-					(size 1.27 1.27)
-				)
-				(hide yes)
-			)
-		)
-		(property "Description" "Hex Inverter"
-			(at 116.84 125.73 0)
-			(effects
-				(font
-					(size 1.27 1.27)
-				)
-				(hide yes)
-			)
-		)
-		(pin "14"
-		)
-		(pin "7"
-		)
-		(pin "1"
-		)
-		(pin "2"
-		)
-		(pin "3"
-		)
-		(pin "4"
-		)
-		(pin "5"
-		)
-		(pin "6"
-		)
-		(pin "8"
-		)
-		(pin "9"
-		)
-		(pin "10"
-		)
-		(pin "11"
-		)
-		(pin "12"
-		)
-		(pin "13"
-		)
-		(instances
-			(project "ecbVera"
-				(path "/d9da1c82-d111-45a9-a5a0-97542a9b1801/915882dc-ec04-4ce2-aae3-dd88b563162b"
-					(reference "U1")
-					(unit 3)
-				)
-			)
-		)
-	)
-	(symbol
 		(lib_id "74xx:74LS32")
 		(at 52.07 67.31 0)
@@
 			)
 		)
-		(property "Value" "74LS04"
+		(property "Value" "74LS06"
 			(at 101.346 128.905 0)
 			(effects
