File: chipselects.kicad_sch (KiCad schematic)
At the start: 12 parts, among them J1 VERA, K2 VERA INTERRUPT SELECT, K3 AUDIO OUT, SW1 VERA ADDR, SW2 Keyboard/Printer, U18 74LS688, U19 74LS688, U20 74LS138, U21 74LS138

Commit message: V1.1
Connections:
- net A2: now also U20.3 (A2), U21.3 (A2)
- net GND: no longer U20.3 (A2), U21.3 (A2)
- net PU1: now also RR2.6 (R5); no longer RR2.10 (R9)
- net B_~{INT}: no longer names the net of RR3.6 (R5)
- net B_~{INT}: no longer K2.1 (Pin_1)
- new net B_/IR6: K2.1 (Pin_1)
Changed lines of the file:
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@@
 	(generator_version "9.0")
 	(paper "A4")
+	(title_block
+		(date "2026-10-24")
+		(rev "V1.1")
+	)
 	(junction
 		(at 44.45 46.99)
@@
 	)
 	(junction
+		(at 165.1 138.43)
+		(diameter 0)
+		(color 0 0 0 0)
+	)
+	(junction
 		(at 135.89 85.09)
 		(diameter 0)
@@
 	)
 	(junction
+		(at 231.14 138.43)
+		(diameter 0)
+		(color 0 0 0 0)
+	)
+	(junction
 		(at 36.83 59.69)
 		(diameter 0)
@@
 	)
 	(no_connect
-		(at 36.83 181.61)
+		(at 72.39 171.45)
 	)
 	(no_connect
-		(at 191.77 128.27)
+		(at 36.83 181.61)
 	)
 	(no_connect
-		(at 36.83 171.45)
+		(at 191.77 128.27)
 	)
 	(no_connect
@@
 	(wire
 		(pts
-			(xy 223.52 130.81) (xy 232.41 130.81)
+			(xy 166.37 130.81) (xy 165.1 130.81)
+		)
+		(stroke
+			(width 0)
+			(type default)
+		)
+	)
+	(wire
+		(pts
+			(xy 231.14 130.81) (xy 231.14 138.43)
 		)
 		(stroke
@@
 	(wire
 		(pts
+			(xy 165.1 138.43) (xy 166.37 138.43)
+		)
+		(stroke
+			(width 0)
+			(type default)
+		)
+	)
+	(wire
+		(pts
 			(xy 134.62 77.47) (xy 135.89 77.47)
 		)
@@
 	(wire
 		(pts
+			(xy 229.87 138.43) (xy 231.14 138.43)
+		)
+		(stroke
+			(width 0)
+			(type default)
+		)
+	)
+	(wire
+		(pts
 			(xy 95.25 69.85) (xy 99.06 69.85)
 		)
@@
 	(wire
 		(pts
+			(xy 165.1 130.81) (xy 165.1 138.43)
+		)
+		(stroke
+			(width 0)
+			(type default)
+		)
+	)
+	(wire
+		(pts
 			(xy 134.62 74.93) (xy 135.89 74.93)
 		)
@@
 	(wire
 		(pts
-			(xy 157.48 130.81) (xy 166.37 130.81)
+			(xy 95.25 62.23) (xy 95.25 64.77)
 		)
 		(stroke
@@
 	(wire
 		(pts
-			(xy 95.25 62.23) (xy 95.25 64.77)
+			(xy 123.19 69.85) (xy 135.89 69.85)
 		)
 		(stroke
@@
 	(wire
 		(pts
-			(xy 123.19 69.85) (xy 135.89 69.85)
+			(xy 232.41 130.81) (xy 231.14 130.81)
 		)
 		(stroke
@@
 	(wire
 		(pts
-			(xy 163.83 138.43) (xy 166.37 138.43)
+			(xy 163.83 138.43) (xy 165.1 138.43)
 		)
 		(stroke
@@
 		)
 	)
+	(global_label "B_{slash}IR6"
+		(shape output)
+		(at 96.52 121.92 0)
+		(fields_autoplaced yes)
+		(effects
+			(font
+				(size 1.27 1.27)
+			)
+			(justify left)
+		)
+		(property "Intersheetrefs" "${INTERSHEET_REFS}"
+			(at 107.8751 121.92 0)
+			(effects
+				(font
+					(size 1.27 1.27)
+				)
+				(justify left)
+				(hide yes)
+			)
+		)
+	)
 	(global_label "B_A7"
 		(shape input)
@@
 	(global_label "PU1"
 		(shape input)
-		(at 36.83 181.61 180)
+		(at 36.83 171.45 180)
 		(fields_autoplaced yes)
 		(effects
@@
 		)
 		(property "Intersheetrefs" "${INTERSHEET_REFS}"
-			(at 30.0348 181.61 0)
+			(at 30.0348 171.45 0)
 			(effects
 				(font
@@
 		)
 	)
-	(global_label "B_~{INT}"
-		(shape input)
-		(at 72.39 171.45 180)
-		(fields_autoplaced yes)
-		(effects
-			(font
-				(size 1.27 1.27)
-			)
-			(justify right)
-		)
-		(property "Intersheetrefs" "${INTERSHEET_REFS}"
-			(at 61.2163 171.45 0)
-			(effects
-				(font
-					(size 1.27 1.27)
-				)
-				(justify right)
-				(hide yes)
-			)
-		)
-	)
 	(global_label "B_~{M1}"
 		(shape input)
@@
 		)
 	)
-	(global_label "B_~{INT}"
-		(shape output)
-		(at 96.52 121.92 0)
-		(fields_autoplaced yes)
-		(effects
-			(font
-				(size 1.27 1.27)
-			)
-			(justify left)
-		)
-		(property "Intersheetrefs" "${INTERSHEET_REFS}"
-			(at 107.6937 121.92 0)
-			(effects
-				(font
-					(size 1.27 1.27)
-				)
-				(justify left)
-				(hide yes)
-			)
-		)
-	)
 	(global_label "A3"
 		(shape input)
@@
 	(global_label "A2"
 		(shape input)
-		(at 231.14 138.43 180)
+		(at 229.87 138.43 180)
 		(fields_autoplaced yes)
 		(effects
@@
 		)
 		(property "Intersheetrefs" "${INTERSHEET_REFS}"
-			(at 225.8567 138.43 0)
+			(at 224.5867 138.43 0)
 			(effects
 				(font
@@
 	)
 	(symbol
-		(lib_id "power:GND")
-		(at 157.48 130.81 0)
-		(unit 1)
-		(exclude_from_sim no)
-		(in_bom yes)
-		(on_board yes)
-		(dnp no)
-		(property "Reference" "#PWR035"
-			(at 157.48 137.16 0)
-			(effects
-				(font
-					(size 1.27 1.27)
-				)
-				(hide yes)
-			)
-		)
-		(property "Value" "GND"
-			(at 157.48 134.366 0)
-			(effects
-				(font
-					(size 1.27 1.27)
-				)
-			)
-		)
-		(property "Footprint" ""
-			(at 157.48 130.81 0)
-			(effects
-				(font
-					(size 1.27 1.27)
-				)
-				(hide yes)
-			)
-		)
-		(property "Datasheet" ""
-			(at 157.48 130.81 0)
-			(effects
-				(font
-					(size 1.27 1.27)
-				)
-				(hide yes)
-			)
-		)
-		(property "Description" "Power symbol creates a global label with name \"GND\" , ground"
-			(at 157.48 130.81 0)
-			(effects
-				(font
-					(size 1.27 1.27)
-				)
-				(hide yes)
-			)
-		)
-		(pin "1"
-		)
-		(instances
-			(project "ecbVera"
-				(path "/d9da1c82-d111-45a9-a5a0-97542a9b1801/06ee56e8-4be0-4ab0-b52c-d9211f2f4421"
-					(reference "#PWR035")
-					(unit 1)
-				)
-			)
-		)
-	)
-	(symbol
 		(lib_id "power:VCC")
 		(at 19.05 82.55 0)
@@
 					(unit 1)
 				)
-			)
-		)
-	)
-	(symbol
-		(lib_id "power:GND")
-		(at 223.52 130.81 0)
-		(unit 1)
-		(exclude_from_sim no)
-		(in_bom yes)
-		(on_board yes)
-		(dnp no)
-		(property "Reference" "#PWR036"
-			(at 223.52 137.16 0)
-			(effects
-				(font
-					(size 1.27 1.27)
-				)
-				(hide yes)
-			)
-		)
-		(property "Value" "GND"
-			(at 223.266 134.366 0)
-			(effects
-				(font
-					(size 1.27 1.27)
-				)
-			)
-		)
-		(property "Footprint" ""
-			(at 223.52 130.81 0)
-			(effects
-				(font
-					(size 1.27 1.27)
-				)
-				(hide yes)
-			)
-		)
-		(property "Datasheet" ""
-			(at 223.52 130.81 0)
-			(effects
-				(font
-					(size 1.27 1.27)
-				)
-				(hide yes)
-			)
-		)
-		(property "Description" "Power symbol creates a global label with name \"GND\" , ground"
-			(at 223.52 130.81 0)
-			(effects
-				(font
-					(size 1.27 1.27)
-				)
-				(hide yes)
-			)
-		)
-		(pin "1"
-		)
-		(instances
-			(project "ecbVera"
-				(path "/d9da1c82-d111-45a9-a5a0-97542a9b1801/06ee56e8-4be0-4ab0-b52c-d9211f2f4421"
-					(reference "#PWR036")
-					(unit 1)
-				)

Commit message: V1.1
Parts:
- added U2: 74LS08, Custom:STD_DDW_DIP14, symbol 74xx:74LS08
- added U4: 74LS32, Custom:STD_DDW_DIP14, symbol 74xx:74LS32
- added U9: 74LS04, Custom:STD_DDW_DIP14, symbol 74xx:74LS04
Connections:
- net ~{VERA}: now also U2.12, U9.3; no longer J1.11 (Pin_11)
- new net: U2.8, U4.10, U4.9
- new net: U4.12, U4.13, U4.8
- new net: U2.10, U2.9, U9.2
- new net: U2.13, U4.11
- new net: U9.1, U9.4
- new net ~{VERASEL}: J1.11 (Pin_11), U2.11
