File: ecbVera.kicad_pcb (KiCad board)
At the start: 2 copper layers, 160 x 100.3 mm, 76 parts, among them J1 VERA, K1 INTERRUPT SELECT, K2 VERA INTERRUPT SELECT, K3 AUDIO OUT, P5 PARALLEL, P6 8 MHz, P7 MOUSE, P8 KEYBOARD, P9 IO PORT, SW1 VERA ADDR, SW2 Keyboard/Printer, U1 74LS04, U10 74LS374, U11 74LS374, U12 74LS244, U13 74LS244, U14 74LS244, U18 74LS688, U19 74LS688, U2 74LS08, U20 74LS138, U21 74LS138, U4 74LS32, U5 74LS245, U6 C96ABC, U7 74LS244, U8 74LS06, U9 74LS04

Commit message: V1.1
Parts:
- U1: value 74LS04 -> 74LS06
Connections:
- K1 pad 1: B_~{INT} -> B_/IR6
- K1 pad 2: Net-(K1-Pin_2) -> PU1
- K2 pad 1: B_~{INT} -> B_/IR6
- RR2 pad 10: PU1 -> unconnected-(RR2-R9-Pad10)
- RR2 pad 6: unconnected-(RR2-R5-Pad6) -> PU1
- RR3 pad 6: B_~{INT} -> unconnected-(RR3-R5-Pad6)
- U1 pad 4: Net-(U1-Pad4) -> PU1
- U1 pad 5: Net-(U1-Pad4) -> unconnected-(U1-Pad5)
- U1 pad 6: Net-(K1-Pin_2) -> unconnected-(U1-Pad6)
- U20 pad 3: GND -> A2
- U21 pad 3: GND -> A2
- U7 pad 11: unconnected-(U7-I0b-Pad11) -> B_A3
- U7 pad 12: unconnected-(U7-O3a-Pad12) -> A4
- U7 pad 8: unconnected-(U7-I3a-Pad8) -> B_A4
- U7 pad 9: unconnected-(U7-O0b-Pad9) -> A3
Routing:
- net B_/IR6: track 0.00 -> 212.9 mm, vias 0 -> 1
- net B_~{INT}: track 208.4 -> 0.00 mm
- net GND: track 977.0 -> 805.4 mm, vias 14 -> 0
- net VCC: track 779.5 -> 662.3 mm, vias 13 -> 0
- net A4: track 0.00 -> 109.5 mm, vias 0 -> 2
- net D6: track 376.5 -> 268.2 mm, vias 10 -> 4
- net A3: track 0.00 -> 100.2 mm, vias 0 -> 1
- net D0: track 364.6 -> 281.4 mm, vias 13 -> 1
- net D5: track 391.2 -> 309.0 mm, vias 9 -> 3
- net Net-(U10-O3): track 182.5 -> 110.5 mm, vias 8 -> 0
- net D2: track 322.4 -> 256.8 mm, vias 9 -> 1
- net D1: track 337.5 -> 279.7 mm, vias 8 -> 3
- net PD2: track 218.9 -> 161.3 mm, vias 7 -> 2
- net Net-(U10-O1): track 181.9 -> 126.7 mm, vias 9 -> 2
- net D7: track 378.0 -> 327.4 mm, vias 9 -> 3
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Other:
- board text added: "VERA INTERFACE VER 1.1"
- board text added: "https://github.com/danwerner21/VERAECB Dan Werner 10/24/2026"
- board text removed: "VERA INTERFACE VER 1"
- board text removed: "https://github.com/danwerner21/VERAECB Dan Werner 10/10/2026"

Commit message: V1.1
Connections:
- J1 pad 11: ~{VERA} -> ~{VERASEL}
- U2 pad 10: unconnected-(U2-Pad10) -> Net-(U2-Pad10)
- U2 pad 11: unconnected-(U2-Pad11) -> ~{VERASEL}
- U2 pad 12: unconnected-(U2-Pad12) -> ~{VERA}
- U2 pad 13: unconnected-(U2-Pad13) -> Net-(U2-Pad13)
- U2 pad 8: unconnected-(U2-Pad8) -> Net-(U2-Pad8)
- U2 pad 9: unconnected-(U2-Pad9) -> Net-(U2-Pad10)
- U4 pad 10: unconnected-(U4-Pad10) -> Net-(U2-Pad8)
- U4 pad 11: unconnected-(U4-Pad11) -> Net-(U2-Pad13)
- U4 pad 12: unconnected-(U4-Pad12) -> Net-(U4-Pad12)
- U4 pad 13: unconnected-(U4-Pad13) -> Net-(U4-Pad12)
- U4 pad 8: unconnected-(U4-Pad8) -> Net-(U4-Pad12)
- U4 pad 9: unconnected-(U4-Pad9) -> Net-(U2-Pad8)
- U9 pad 1: unconnected-(U9-Pad1) -> Net-(U9-Pad1)
- U9 pad 2: unconnected-(U9-Pad2) -> Net-(U2-Pad10)
- U9 pad 3: unconnected-(U9-Pad3) -> ~{VERA}
- U9 pad 4: unconnected-(U9-Pad4) -> Net-(U9-Pad1)
Routing:
- net VCC: track 662.3 -> 796.4 mm, vias 0 -> 7
- net GND: track 805.4 -> 922.0 mm, vias 0 -> 8
- net Net-(U2-Pad10): track 0.00 -> 114.3 mm, vias 0 -> 1
- net ~{VERASEL}: track 0.00 -> 105.2 mm, vias 0 -> 1
- net Net-(U2-Pad8): track 0.00 -> 72.8 mm, vias 0 -> 2
- net Net-(U2-Pad13): track 0.00 -> 62.0 mm, vias 0 -> 4
- net D2: track 256.8 -> 312.3 mm, vias 1 -> 6
- net ~{STROBE}: track 213.5 -> 170.6 mm
- net D6: track 268.2 -> 304.2 mm, vias 4 -> 7
- net Net-(U10-O2): track 114.9 -> 145.1 mm, vias 0 -> 5
- net A4: track 109.5 -> 138.8 mm
- net D1: track 279.7 -> 308.3 mm, vias 3 -> 4
- net A0: track 200.8 -> 227.9 mm
- net B_~{M1}: track 128.0 -> 102.1 mm, vias 1 -> 3
- net B_~{IR0}: track 223.6 -> 198.3 mm, vias 0 -> 1
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