File: ecbVera.kicad_sch (KiCad schematic)
At the start: 30 parts, among them U1 74LS04, U2 74LS08, U4 74LS32, U8 74LS06, U9 74LS04

Commit message: V1.1
Parts:
- added unit 3 of U1
- U1: value 74LS04 -> 74LS06
Connections:
- no-connect marks 21 -> 23
Changed lines of the file:
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@@
 	(generator_version "9.0")
 	(paper "A4")
+	(title_block
+		(date "2026-10-24")
+		(rev "V1.1")
+	)
 	(text "SPARE"
 		(exclude_from_sim no)
@@
 	)
 	(no_connect
+		(at 86.36 78.74)
+	)
+	(no_connect
+		(at 71.12 78.74)
+	)
+	(no_connect
 		(at 50.8 69.85)
 	)
@@
 		(dnp no)
 		(property "Reference" "U1"
-			(at 260.223 113.919 0)
+			(at 255.27 115.316 0)
 			(effects
 				(font
@@
 			)
 		)
-		(property "Value" "74LS04"
-			(at 260.096 120.015 0)
+		(property "Value" "74LS06"
+			(at 255.016 118.11 0)
 			(effects
 				(font
@@
 				)
 			)
+		)
+	)
+	(symbol
+		(lib_id "74xx:74LS04")
+		(at 78.74 78.74 0)
+		(unit 3)
+		(exclude_from_sim no)
+		(in_bom yes)
+		(on_board yes)
+		(dnp no)
+		(property "Reference" "U1"
+			(at 77.724 78.994 0)
+			(effects
+				(font
+					(size 1.524 1.524)
+				)
+			)
+		)
+		(property "Value" "74LS06"
+			(at 83.566 81.915 0)
+			(effects
+				(font
+					(size 1.524 1.524)
+				)
+			)
+		)
+		(property "Footprint" "Custom:STD_DDW_DIP14"
+			(at 78.74 78.74 0)
+			(effects
+				(font
+					(size 1.27 1.27)
+				)
+				(hide yes)
+			)
+		)
+		(property "Datasheet" "http://www.ti.com/lit/gpn/sn74LS04"
+			(at 78.74 78.74 0)
+			(effects
+				(font
+					(size 1.27 1.27)
+				)
+				(hide yes)
+			)
+		)
+		(property "Description" "Hex Inverter"
+			(at 78.74 78.74 0)
+			(effects
+				(font
+					(size 1.27 1.27)
+				)
+				(hide yes)
+			)
+		)
+		(pin "14"
+		)
+		(pin "7"
+		)
+		(pin "1"
+		)
+		(pin "2"
+		)
+		(pin "3"
+		)
+		(pin "4"
+		)
+		(pin "5"
+		)
+		(pin "6"
+		)
+		(pin "8"
+		)
+		(pin "9"
+		)
+		(pin "10"
+		)
+		(pin "11"
+		)
+		(pin "12"
+		)
+		(pin "13"
+		)
+		(instances
+			(project "ecbVera"
+				(path "/d9da1c82-d111-45a9-a5a0-97542a9b1801"
+					(reference "U1")
+					(unit 3)
+				)
+			)

Commit message: V1.1
Parts:
- removed unit 3 of U2
- removed unit 4 of U2
- removed unit 3 of U4
- removed unit 4 of U4
- removed unit 2 of U9
- removed unit 1 of U9
Connections:
- no-connect marks 23 -> 7
